File: rucheb.kicad_sch (KiCad schematic)
At the start: 23 parts, among them IC1 CN3791, J1 Conn_01x02, Q1 AO3401A

Commit message: Correction cartouche schéma
Other:
- company: (none) -> Ratamuse
- title: Testboard V2.3b -> Open_beehive_scale_board
Changed lines of the file:
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@@
   (paper "A4")
   (title_block
-    (title "Testboard V2.3b")
+    (title "Open_beehive_scale_board")
     (date "2021-12-11")
+    (rev "V0.1")
+    (company "Ratamuse")
   )
   (junction (at 215.9 41.91) (diameter 0) (color 0 0 0 0)
