File: rucheb.kicad_sch (KiCad schematic)
At the start: 23 parts, among them IC1 CN3791, J1 Conn_01x02, Q1 AO3401A

Commit message: V0.2
Other:
- note added: "1/The maximum power point voltage is decided by the following equation: VMPPT=1.205x(1+R5/R4) 2/Charge current setting The full-scale charge current, namely the charge current in constant current mode, is decided by the following formula: ICH= 120mV/R6 500mA=0.24 ohm 250mA=0.48 ohm 125mA=0.96 ohm"
- note removed: "1/The maximum power point voltage is decided by the following equation: VMPPT=1.205x(1+R23/R27) 2/Charge current setting The full-scale charge current, namely the charge current in constant current mode, is decided by the following formula: ICH= 120mV/R28 500mA=0.24 ohm 250mA=0.48 ohm 125mA=0.96 ohm"
Changed lines of the file:
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@@
     (stroke (width 0) (type default) (color 0 0 0 0))
   )
-  (text "1/The maximum power point voltage is decided\nby the following equation:\n\nVMPPT=1.205x(1+R23/R27)\n\n2/Charge current setting\n\nThe full-scale charge current, namely the charge current in \nconstant current mode, is decided by the following formula:\n\nICH= 120mV/R28\n\n500mA=0.24 ohm\n250mA=0.48 ohm\n125mA=0.96 ohm"
+  (text "1/The maximum power point voltage is decided\nby the following equation:\n\nVMPPT=1.205x(1+R5/R4)\n\n2/Charge current setting\n\nThe full-scale charge current, namely the charge current in \nconstant current mode, is decided by the following formula:\n\nICH= 120mV/R6\n\n500mA=0.24 ohm\n250mA=0.48 ohm\n125mA=0.96 ohm"
     (at 147.32 133.35 0)
     (effects (font (size 1.27 1.27)) (justify left bottom))
